File: Electronics/Supply-Board/Supply-Board.kicad_pcb (KiCad board)
At the start: 2 copper layers, 160 x 99.5 mm, 91 parts, among them J1 DB25_Female_MountingHoles, J2 PE, J3 L, J4 N, T1 VC 5,0/2/15, T2 VC 5,0/2/18, U1 LM317, U2 LM337, U3 LM317, U4 LM337, U5 traco_TSR_0.5-2433, U6 LM75C

Commit message: Power Supply Design Requirements
Connections:
- J1 pad 25: Net-(J1-Pad25) -> unconnected-(J1-P25-Pad25)
- U6 pad 3: Net-(U6-Pad3) -> unconnected-(U6-O.S.-Pad3)
Routing:
- net /digital_gnd: track 175.5 -> 180.2 mm
- net /stepper_9V: track 150.1 -> 152.6 mm
Other:
- net class Default removed
- board text added: "~230V"
- board text removed: "STM Supply Board V1 J.H. 2019"
- board text removed: "~~230V"
