File: Electronics/Tunnelling-Amp/Tunnelling-Amp.kicad_pcb (KiCad board)
At the start: 2 copper layers, 49.8 x 19.8 mm, 19 parts, among them J1 RF_Shield_Two_Pieces, U1 ADA4637-1

Commit message: Power Supply Design Requirements
Other:
- net class Default removed
